Commit message: Made a victor with only the right arm

File: urdf/iiwa7.xacro (robot description, xacro)
@@ -2,9 +2,9 @@
 <robot xmlns:xacro="http://www.ros.org/wiki/xacro">
     <!-- Import all Gazebo-customization elements, including Gazebo colors -->
-    <xacro:include filename="$(find victor_description)/urdf/iiwa.gazebo.xacro"/>
+    <xacro:include filename="$(find gpu_voxel_planning)/urdf/iiwa.gazebo.xacro"/>
     <!-- Import Transmissions -->
-    <xacro:include filename="$(find victor_description)/urdf/iiwa.transmission.xacro"/>
+    <xacro:include filename="$(find gpu_voxel_planning)/urdf/iiwa.transmission.xacro"/>
     <!-- Include Utilities -->
-    <xacro:include filename="$(find victor_description)/urdf/utilities.xacro"/>
+    <xacro:include filename="$(find gpu_voxel_planning)/urdf/utilities.xacro"/>
     <!-- some constants -->
     <xacro:property name="safety_controller_k_pos" value="100"/>
@@ -29,5 +29,5 @@
                 <origin xyz="0 0 0" rpy="0 0 0"/>
                 <geometry>
-                    <mesh filename="package://victor_description/meshes/iiwa7/visual/link_0.stl"/>
+                    <mesh filename="package://gpu_voxel_planning/meshes/iiwa7/visual/link_0.stl"/>
                 </geometry>
                 <material name="Grey"/>
@@ -36,5 +36,5 @@
                 <origin xyz="0 0 0" rpy="0 0 0"/>
                 <geometry>
-                    <mesh filename="package://victor_description/meshes/iiwa7/collision/link_0.stl"/>
+                    <mesh filename="package://gpu_voxel_planning/meshes/iiwa7/collision/link_0.stl"/>
                 </geometry>
                 <material name="Grey"/>
@@ -70,5 +70,5 @@
                 <origin xyz="0 0 0.0075" rpy="0 0 0"/>
                 <geometry>
-                    <mesh filename="package://victor_description/meshes/iiwa7/visual/link_1.stl"/>
+                    <mesh filename="package://gpu_voxel_planning/meshes/iiwa7/visual/link_1.stl"/>
                 </geometry>
                 <material name="Orange"/>
@@ -77,5 +77,5 @@
                 <origin xyz="0 0 0.0075" rpy="0 0 0"/>
                 <geometry>
-                    <mesh filename="package://victor_description/meshes/iiwa7/collision/link_1.stl"/>
+                    <mesh filename="package://gpu_voxel_planning/meshes/iiwa7/collision/link_1.stl"/>
                 </geometry>
                 <material name="Orange"/>
@@ -104,12 +104,12 @@
                 <origin xyz="0 0 0" rpy="0 0 0"/>
                 <geometry>
-                    <mesh filename="package://victor_description/meshes/iiwa7/visual/link_2.stl"/>
-                </geometry>
-                <material name="Orange"/>
-            </visual>
-            <collision>
-                <origin xyz="0 0 0" rpy="0 0 0"/>
-                <geometry>
-                    <mesh filename="package://victor_description/meshes/iiwa7/collision/link_2.stl"/>
+                    <mesh filename="package://gpu_voxel_planning/meshes/iiwa7/visual/link_2.stl"/>
+                </geometry>
+                <material name="Orange"/>
+            </visual>
+            <collision>
+                <origin xyz="0 0 0" rpy="0 0 0"/>
+                <geometry>
+                    <mesh filename="package://gpu_voxel_planning/meshes/iiwa7/collision/link_2.stl"/>
                 </geometry>
                 <material name="Orange"/>
@@ -138,5 +138,5 @@
                 <origin xyz="0 0 -0.026" rpy="0 0 0"/>
                 <geometry>
-                    <mesh filename="package://victor_description/meshes/iiwa7/visual/link_3.stl"/>
+                    <mesh filename="package://gpu_voxel_planning/meshes/iiwa7/visual/link_3.stl"/>
                 </geometry>
                 <material name="Orange"/>
@@ -145,5 +145,5 @@
                 <origin xyz="0 0 -0.026" rpy="0 0 0"/>
                 <geometry>
-                    <mesh filename="package://victor_description/meshes/iiwa7/collision/link_3.stl"/>
+                    <mesh filename="package://gpu_voxel_planning/meshes/iiwa7/collision/link_3.stl"/>
                 </geometry>
                 <material name="Orange"/>
@@ -172,12 +172,12 @@
                 <origin xyz="0 0 0" rpy="0 0 0"/>
                 <geometry>
-                    <mesh filename="package://victor_description/meshes/iiwa7/visual/link_4.stl"/>
-                </geometry>
-                <material name="Orange"/>
-            </visual>
-            <collision>
-                <origin xyz="0 0 0" rpy="0 0 0"/>
-                <geometry>
-                    <mesh filename="package://victor_description/meshes/iiwa7/collision/link_4.stl"/>
+                    <mesh filename="package://gpu_voxel_planning/meshes/iiwa7/visual/link_4.stl"/>
+                </geometry>
+                <material name="Orange"/>
+            </visual>
+            <collision>
+                <origin xyz="0 0 0" rpy="0 0 0"/>
+                <geometry>
+                    <mesh filename="package://gpu_voxel_planning/meshes/iiwa7/collision/link_4.stl"/>
                 </geometry>
                 <material name="Orange"/>
@@ -206,5 +206,5 @@
                 <origin xyz="0 0 -0.026" rpy="0 0 0"/>
                 <geometry>
-                    <mesh filename="package://victor_description/meshes/iiwa7/visual/link_5.stl"/>
+                    <mesh filename="package://gpu_voxel_planning/meshes/iiwa7/visual/link_5.stl"/>
                 </geometry>
                 <material name="Orange"/>
@@ -213,5 +213,5 @@
                 <origin xyz="0 0 -0.026" rpy="0 0 0"/>
                 <geometry>
-                    <mesh filename="package://victor_description/meshes/iiwa7/collision/link_5.stl"/>
+                    <mesh filename="package://gpu_voxel_planning/meshes/iiwa7/collision/link_5.stl"/>
                 </geometry>
                 <material name="Orange"/>
@@ -240,12 +240,12 @@
                 <origin xyz="0 0 0" rpy="0 0 0"/>
                 <geometry>
-                    <mesh filename="package://victor_description/meshes/iiwa7/visual/link_6.stl"/>
-                </geometry>
-                <material name="Orange"/>
-            </visual>
-            <collision>
-                <origin xyz="0 0 0" rpy="0 0 0"/>
-                <geometry>
-                    <mesh filename="package://victor_description/meshes/iiwa7/collision/link_6.stl"/>
+                    <mesh filename="package://gpu_voxel_planning/meshes/iiwa7/visual/link_6.stl"/>
+                </geometry>
+                <material name="Orange"/>
+            </visual>
+            <collision>
+                <origin xyz="0 0 0" rpy="0 0 0"/>
+                <geometry>
+                    <mesh filename="package://gpu_voxel_planning/meshes/iiwa7/collision/link_6.stl"/>
                 </geometry>
                 <material name="Orange"/>
@@ -274,5 +274,5 @@
                 <origin xyz="0 0 -0.0005" rpy="0 0 0"/>
                 <geometry>
-                    <mesh filename="package://victor_description/meshes/iiwa7/visual/link_7_electric.stl"/>
+                    <mesh filename="package://gpu_voxel_planning/meshes/iiwa7/visual/link_7_electric.stl"/>
                 </geometry>
                 <material name="Grey"/>
@@ -281,5 +281,5 @@
                 <origin xyz="0 0 -0.0005" rpy="0 0 0"/>
                 <geometry>
-                    <mesh filename="package://victor_description/meshes/iiwa7/collision/link_7_electric.stl"/>
+                    <mesh filename="package://gpu_voxel_planning/meshes/iiwa7/collision/link_7_electric.stl"/>
                 </geometry>
                 <material name="Grey"/>
