Commit message: modify urdf to allow for right and left arms separately

File: urdf/baxter_pedestal.xacro (robot description, xacro)
@@ -20,5 +20,5 @@
                 <origin rpy="0 0 0" xyz="0 0 0.9245"/>
                 <geometry>
-                    <mesh filename="package://victor_description/meshes/baxter_pedestal/pedestal_collision.stl"/>
+                    <mesh filename="package://victor_description/meshes/baxter_pedestal/pedestal_visual.stl"/>
                 </geometry>
                 <material name="DarkGray"/>

File: urdf/iiwa7.xacro (robot description, xacro)
@@ -34,5 +34,5 @@
             </visual>
             <collision>
-                <origin xyz="0 0 0" rpy="0 0 0"/>
+                <origin xyz="0 0 0.05" rpy="0 0 0"/>
                 <geometry>
                     <mesh filename="package://gpu_voxel_planning/meshes/iiwa7/collision/link_0.stl"/>

File: urdf/victor_left_arm_and_body.urdf (robot description, URDF)
Before this commit: robot victor, 34 links, 33 joints
Links:
- removed link victor_right_arm_flange
- removed link victor_right_arm_flange_kuka
- removed link victor_right_arm_link_0
- removed link victor_right_arm_link_1
- removed link victor_right_arm_link_2
- removed link victor_right_arm_link_3
- removed link victor_right_arm_link_4
- removed link victor_right_arm_link_5
- removed link victor_right_arm_link_6
- removed link victor_right_arm_link_7
- removed link victor_right_arm_world_frame_kuka
- removed link victor_right_gripper_fingerA_base
- removed link victor_right_gripper_fingerA_dist
- removed link victor_right_gripper_fingerA_med
- removed link victor_right_gripper_fingerA_prox
- removed link victor_right_gripper_fingerB_base
- removed link victor_right_gripper_fingerB_dist
- removed link victor_right_gripper_fingerB_med
- removed link victor_right_gripper_fingerB_prox
- removed link victor_right_gripper_fingerC_base
- removed link victor_right_gripper_fingerC_dist
- removed link victor_right_gripper_fingerC_med
- removed link victor_right_gripper_fingerC_prox
- removed link victor_right_gripper_mounting_bracket
- removed link victor_right_gripper_palm
- removed link victor_right_gripper_palm_surface
- removed link victor_right_gripper_palm_surface_kuka
- added link victor_left_arm_flange
- added link victor_left_arm_flange_kuka
- added link victor_left_arm_link_0, mass 5; collision mesh filename=package://gpu_voxel_planning/meshes/iiwa7/collision/link_0.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; visual mesh filename=package://gpu_voxel_planning/meshes/iiwa7/visual/link_0.stl
- added link victor_left_arm_link_1, mass 3.4525; collision mesh filename=package://gpu_voxel_planning/meshes/iiwa7/collision/link_1.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; visual mesh filename=package://gpu_voxel_planning/meshes/iiwa7/visual/link_1.stl
- added link victor_left_arm_link_2, mass 3.4821; collision mesh filename=package://gpu_voxel_planning/meshes/iiwa7/collision/link_2.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; visual mesh filename=package://gpu_voxel_planning/meshes/iiwa7/visual/link_2.stl
- added link victor_left_arm_link_3, mass 4.05623; collision mesh filename=package://gpu_voxel_planning/meshes/iiwa7/collision/link_3.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; visual mesh filename=package://gpu_voxel_planning/meshes/iiwa7/visual/link_3.stl
- added link victor_left_arm_link_4, mass 3.4822; collision mesh filename=package://gpu_voxel_planning/meshes/iiwa7/collision/link_4.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; visual mesh filename=package://gpu_voxel_planning/meshes/iiwa7/visual/link_4.stl
- added link victor_left_arm_link_5, mass 2.1633; collision mesh filename=package://gpu_voxel_planning/meshes/iiwa7/collision/link_5.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; visual mesh filename=package://gpu_voxel_planning/meshes/iiwa7/visual/link_5.stl
- added link victor_left_arm_link_6, mass 2.3466; collision mesh filename=package://gpu_voxel_planning/meshes/iiwa7/collision/link_6.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; visual mesh filename=package://gpu_voxel_planning/meshes/iiwa7/visual/link_6.stl
- added link victor_left_arm_link_7, mass 3.129; collision mesh filename=package://gpu_voxel_planning/meshes/iiwa7/collision/link_7_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; visual mesh filename=package://gpu_voxel_planning/meshes/iiwa7/visual/link_7_ele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
- added link victor_left_arm_world_frame_kuka
- added link victor_left_gripper_fingerA_base, mass 1; collision mesh filename=package://victor_description/meshes/robotiq_3finger/finger_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; visual mesh filename=package://victor_description/meshes/robotiq_3finger/finger_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
- added link victor_left_gripper_fingerA_dist, mass 1; collision mesh filename=package://victor_description/meshes/robotiq_3finger/finger_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; visual mesh filename=package://victor_description/meshes/robotiq_3finger/finger_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
- added link victor_left_gripper_fingerA_med, mass 1; collision mesh filename=package://victor_description/meshes/robotiq_3finger/finger_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; visual mesh filename=package://victor_description/meshes/robotiq_3finger/finger_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
- added link victor_left_gripper_fingerA_prox, mass 1; collision mesh filename=package://victor_description/meshes/robotiq_3finger/finger_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; visual mesh filename=package://victor_description/meshes/robotiq_3finger/finger_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
- added link victor_left_gripper_fingerB_base, mass 1; collision mesh filename=package://victor_description/meshes/robotiq_3finger/finger_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; visual mesh filename=package://victor_description/meshes/robotiq_3finger/finger_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
- added link victor_left_gripper_fingerB_dist, mass 1; collision mesh filename=package://victor_description/meshes/robotiq_3finger/finger_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; visual mesh filename=package://victor_description/meshes/robotiq_3finger/finger_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
- added link victor_left_gripper_fingerB_med, mass 1; collision mesh filename=package://victor_description/meshes/robotiq_3finger/finger_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; visual mesh filename=package://victor_description/meshes/robotiq_3finger/finger_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
- added link victor_left_gripper_fingerB_prox, mass 1; collision mesh filename=package://victor_description/meshes/robotiq_3finger/finger_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; visual mesh filename=package://victor_description/meshes/robotiq_3finger/finger_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
- added link victor_left_gripper_fingerC_base, mass 1; collision mesh filename=package://victor_description/meshes/robotiq_3finger/finger_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; visual mesh filename=package://victor_description/meshes/robotiq_3finger/finger_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
- added link victor_left_gripper_fingerC_dist, mass 1; collision mesh filename=package://victor_description/meshes/robotiq_3finger/finger_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; visual mesh filename=package://victor_description/meshes/robotiq_3finger/finger_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
- added link victor_left_gripper_fingerC_med, mass 1; collision mesh filename=package://victor_description/meshes/robotiq_3finger/finger_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; visual mesh filename=package://victor_description/meshes/robotiq_3finger/finger_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
- added link victor_left_gripper_fingerC_prox, mass 1; collision mesh filename=package://victor_description/meshes/robotiq_3finger/finger_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; visual mesh filename=package://victor_description/meshes/robotiq_3finger/finger_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
- added link victor_left_gripper_mounting_bracket; collision mesh filename=package://victor_description/meshes/robotiq_3finger/kuka_to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; visual mesh filename=package://victor_description/meshes/robotiq_3finger/kuka_to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
- added link victor_left_gripper_palm, mass 1; collision mesh filename=package://victor_description/meshes/robotiq_3finger/palm_co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; visual mesh filename=package://victor_description/meshes/robotiq_3finger/palm_vi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
- added link victor_left_gripper_palm_surface
- added link victor_left_gripper_palm_surface_kuka
- link victor_base_plate: geometry collision mesh filename=package://victor_description/meshes/torso/torso_visual.stl; visual mesh filename=package://victor_description/meshes/torso/torso_visual.stl
- link victor_pedestal: geometry collision mesh filename=package://victor_description/meshes/baxter_pedestal/pedesta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; visual mesh filename=package://victor_description/meshes/baxter_pedestal/pedesta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
Joints:
- removed joint victor_joint_right_arm_world_frame_kuka
- removed joint victor_right_arm_flange_kuka_joint
- removed joint victor_right_arm_flange_victor_right_joint
- removed joint victor_right_arm_joint_1
- removed joint victor_right_arm_joint_2
- removed joint victor_right_arm_joint_3
- removed joint victor_right_arm_joint_4
- removed joint victor_right_arm_joint_5
- removed joint victor_right_arm_joint_6
- removed joint victor_right_arm_joint_7
- removed joint victor_right_arm_joint_flange
- removed joint victor_right_arm_mount_victor_right_arm_joint
- removed joint victor_right_gripper_fingerA_joint_2
- removed joint victor_right_gripper_fingerA_joint_3
- removed joint victor_right_gripper_fingerA_joint_4
- removed joint victor_right_gripper_fingerA_knuckle
- removed joint victor_right_gripper_fingerB_joint_2
- removed joint victor_right_gripper_fingerB_joint_3
- removed joint victor_right_gripper_fingerB_joint_4
- removed joint victor_right_gripper_fingerB_knuckle
- removed joint victor_right_gripper_fingerC_joint_2
- removed joint victor_right_gripper_fingerC_joint_3
- removed joint victor_right_gripper_fingerC_joint_4
- removed joint victor_right_gripper_fingerC_knuckle
- removed joint victor_right_gripper_palm_joint
- removed joint victor_right_gripper_palm_surface_joint
- removed joint victor_right_gripper_palm_surface_kuka_joint
- added joint victor_joint_left_arm_world_frame_kuka: type fixed, parent victor_left_arm_mount, child victor_left_arm_world_frame_kuka, origin xyz=0 0 0 rpy=1.57079632679 0 0
- added joint victor_left_arm_flange_kuka_joint: type fixed, parent victor_left_arm_flange, child victor_left_arm_flange_kuka, origin xyz=0 0 0 rpy=0 0 0
- added joint victor_left_arm_flange_victor_left_joint: type fixed, parent victor_left_arm_flange, child victor_left_gripper_mounting_bracket, origin xyz=0 0 0 rpy=0 0 0
- added joint victor_left_arm_joint_1: type revolute, parent victor_left_arm_link_0, child victor_left_arm_link_1, origin xyz=0 0 0.15 rpy=0 0 0, axis 0 0 1, limit lower=-2.96705972839 upper=2.96705972839 effort=300 velocity=10
- added joint victor_left_arm_joint_2: type revolute, parent victor_left_arm_link_1, child victor_left_arm_link_2, origin xyz=0 0 0.19 rpy=1.57079632679   0 3.14159265359, axis 0 0 1, limit lower=-2.09439510239 upper=2.09439510239 effort=300 velocity=10
- added joint victor_left_arm_joint_3: type revolute, parent victor_left_arm_link_2, child victor_left_arm_link_3, origin xyz=0 0.21 0 rpy=1.57079632679 0 3.14159265359, axis 0 0 1, limit lower=-2.96705972839 upper=2.96705972839 effort=300 velocity=10
- added joint victor_left_arm_joint_4: type revolute, parent victor_left_arm_link_3, child victor_left_arm_link_4, origin xyz=0 0 0.19 rpy=1.57079632679 0 0, axis 0 0 1, limit lower=-2.09439510239 upper=2.09439510239 effort=300 velocity=10
- added joint victor_left_arm_joint_5: type revolute, parent victor_left_arm_link_4, child victor_left_arm_link_5, origin xyz=0 0.21 0 rpy=-1.57079632679 3.14159265359 0, axis 0 0 1, limit lower=-2.96705972839 upper=2.96705972839 effort=300 velocity=10
- added joint victor_left_arm_joint_6: type revolute, parent victor_left_arm_link_5, child victor_left_arm_link_6, origin xyz=0 0.06070 0.19 rpy=1.57079632679 0 0, axis 0 0 1, limit lower=-2.09439510239 upper=2.09439510239 effort=300 velocity=10
- added joint victor_left_arm_joint_7: type revolute, parent victor_left_arm_link_6, child victor_left_arm_link_7, origin xyz=0 0.081 0.06070 rpy=-1.57079632679 3.14159265359 0, axis 0 0 1, limit lower=-3.05432619099 upper=3.05432619099 effort=300 velocity=10
- added joint victor_left_arm_joint_flange: type fixed, parent victor_left_arm_link_7, child victor_left_arm_flange, origin xyz=0 0 0.045 rpy=0 0 0
- added joint victor_left_arm_mount_victor_left_arm_joint: type fixed, parent victor_left_arm_mount, child victor_left_arm_link_0, origin xyz=0 0 0 rpy=0 0 0
- added joint victor_left_gripper_fingerA_joint_2: type revolute, parent victor_left_gripper_fingerA_base, child victor_left_gripper_fingerA_prox, origin xyz=0.02225000 0 0.02151380 rpy=0 0.610865238198 0, axis 0 -1 0, limit lower=-1 upper=1 effort=300 velocity=10
- added joint victor_left_gripper_fingerA_joint_3: type revolute, parent victor_left_gripper_fingerA_prox, child victor_left_gripper_fingerA_med, origin xyz=0 0 0.05715000 rpy=0 0 0, axis 0 -1 0, limit lower=-1 upper=1 effort=300 velocity=10
- added joint victor_left_gripper_fingerA_joint_4: type revolute, parent victor_left_gripper_fingerA_med, child victor_left_gripper_fingerA_dist, origin xyz=0 0 0.03810000 rpy=0 -0.436332312999 0, axis 0 -1 0, limit lower=-1 upper=1 effort=300 velocity=10
- added joint victor_left_gripper_fingerA_knuckle: type fixed, parent victor_left_gripper_palm, child victor_left_gripper_fingerA_base, origin xyz=0.02225040 0 0.06111875 rpy=0 0 0
- added joint victor_left_gripper_fingerB_joint_2: type revolute, parent victor_left_gripper_fingerB_base, child victor_left_gripper_fingerB_prox, origin xyz=0.02225000 0 0.02151380 rpy=0 0.610865238198 0, axis 0 -1 0, limit lower=-1 upper=1 effort=300 velocity=10
- added joint victor_left_gripper_fingerB_joint_3: type revolute, parent victor_left_gripper_fingerB_prox, child victor_left_gripper_fingerB_med, origin xyz=0 0 0.05715000 rpy=0 0 0, axis 0 -1 0, limit lower=-1 upper=1 effort=300 velocity=10
- added joint victor_left_gripper_fingerB_joint_4: type revolute, parent victor_left_gripper_fingerB_med, child victor_left_gripper_fingerB_dist, origin xyz=0 0 0.03810000 rpy=0 -0.436332312999 0, axis 0 -1 0, limit lower=-1 upper=1 effort=300 velocity=10
- added joint victor_left_gripper_fingerB_knuckle: type revolute, parent victor_left_gripper_palm, child victor_left_gripper_fingerB_base, origin xyz=-0.02230120 0.03651250 0.06111875 rpy=0 0 3.14159265359, axis -1 0 0, limit lower=-0.279252680319 upper=0.174532925199 effort=300 velocity=10
- added joint victor_left_gripper_fingerC_joint_2: type revolute, parent victor_left_gripper_fingerC_base, child victor_left_gripper_fingerC_prox, origin xyz=0.02225000 0 0.02151380 rpy=0 0.610865238198 0, axis 0 -1 0, limit lower=-1 upper=1 effort=300 velocity=10
- added joint victor_left_gripper_fingerC_joint_3: type revolute, parent victor_left_gripper_fingerC_prox, child victor_left_gripper_fingerC_med, origin xyz=0 0 0.05715000 rpy=0 0 0, axis 0 -1 0, limit lower=-1 upper=1 effort=300 velocity=10
- added joint victor_left_gripper_fingerC_joint_4: type revolute, parent victor_left_gripper_fingerC_med, child victor_left_gripper_fingerC_dist, origin xyz=0 0 0.03810000 rpy=0 -0.436332312999 0, axis 0 -1 0, limit lower=-1 upper=1 effort=300 velocity=10
- added joint victor_left_gripper_fingerC_knuckle: type revolute, parent victor_left_gripper_palm, child victor_left_gripper_fingerC_base, origin xyz=-0.02230120 -0.03651250 0.06111875 rpy=0 0 3.14159265359, axis 1 0 0, limit lower=-0.279252680319 upper=0.174532925199 effort=300 velocity=10
- added joint victor_left_gripper_palm_joint: type fixed, parent victor_left_gripper_mounting_bracket, child victor_left_gripper_palm, origin xyz=0 0 0.02705 rpy=0 0 0.785398163397
- added joint victor_left_gripper_palm_surface_joint: type fixed, parent victor_left_gripper_palm, child victor_left_gripper_palm_surface, origin xyz=0 0 0.092075 rpy=0 0 0
- added joint victor_left_gripper_palm_surface_kuka_joint: type fixed, parent victor_left_gripper_palm_surface, child victor_left_gripper_palm_surface_kuka, origin xyz=0 0 0 rpy=0 0 0

File: urdf/victor_torso.xacro (robot description, xacro)
@@ -17,8 +17,8 @@
             </visual>
             <collision>
-                <origin xyz="0 0 0.2" rpy="0 0 0"/>
+                <origin xyz="0 0 0" rpy="0 0 0"/>
                 <geometry>
-                    <!--<mesh filename="package://victor_description/meshes/torso_visual_model.stl"/>-->
-                    <cylinder length="0.7" radius="0.2"/>
+                    <mesh filename="package://victor_description/meshes/torso/torso_visual.stl"/>
+                    <!-- <cylinder length="0.7" radius="0.2"/> -->
                 </geometry>
                 <material name="LightGrey"/>
@@ -32,12 +32,12 @@
         </joint>
         <link name="${robot_name}_left_arm_mount">
-            <collision>
-                <origin xyz="0 0 -0.013" rpy="0 0 0"/>
-                <geometry>
-                    <!--<mesh filename="package://victor_description/meshes/torso_visual_model.stl"/>-->
-                    <box size="0.31 0.31 0.032"/>
-                </geometry>
-                <material name="LightGrey"/>
-            </collision>
+            <!-- <collision> -->
+            <!--     <origin xyz="0 0 -0.013" rpy="0 0 0"/> -->
+            <!--     <geometry> -->
+            <!--         <!-\-<mesh filename="package://victor_description/meshes/torso_visual_model.stl"/>-\-> -->
+            <!--         <!-\- <box size="0.31 0.31 0.032"/> -\-> -->
+            <!--     </geometry> -->
+            <!--     <material name="LightGrey"/> -->
+            <!-- </collision> -->
         </link>
         <joint name="${robot_name}_right_arm_mount_joint" type="fixed">
@@ -48,12 +48,12 @@
         </joint>
         <link name="${robot_name}_right_arm_mount">
-            <collision>
-                <origin xyz="0 0 -0.013" rpy="0 0 0"/>
-                <geometry>
-                    <!--<mesh filename="package://victor_description/meshes/torso_visual_model.stl"/>-->
-                    <box size="0.31 0.31 0.032"/>
-                </geometry>
-                <material name="LightGrey"/>
-            </collision>
+            <!-- <collision> -->
+            <!--     <origin xyz="0 0 -0.013" rpy="0 0 0"/> -->
+            <!--     <geometry> -->
+            <!--         <mesh filename="package://victor_description/meshes/torso_visual_model.stl"/> -->
+            <!--         <!-\- <box size="0.31 0.31 0.032"/> -\-> -->
+            <!--     </geometry> -->
+            <!--     <material name="LightGrey"/> -->
+            <!-- </collision> -->
         </link>
     </xacro:macro>

File: urdf/victor_torso_no_links.xacro (robot description, xacro)
@@ -5,5 +5,5 @@
             <parent link="${parent}"/>
             <child link="${robot_name}_base_plate"/>
-            <origin xyz="0 0 0.2" rpy="0 0 0"/>
+            <origin xyz="0 0 0" rpy="0 0 0"/>
             <axis xyz="0 0 1"/>
         </joint>
