Commit message: Just made video on robot

File: urdf/victor_right_arm_with_rod.urdf (robot description, URDF)
Before this commit: robot victor_with_rod, 35 links, 34 joints
Links:
- link rod: geometry collision cylinder length=0.234 radius=0.065
Joints:
- joint rod_joint: origin xyz=0 0 0.1 rpy=1.57 0 0 -> xyz=0 0 0.15 rpy=1.57 0 0
- joint victor_right_gripper_fingerA_joint_2: limit lower=-1 upper=1 effort=300 velocity=10 -> lower=0 upper=1.2217304763960307 effort=300 velocity=10
- joint victor_right_gripper_fingerB_joint_2: limit lower=-1 upper=1 effort=300 velocity=10 -> lower=0 upper=1.2217304763960307 effort=300 velocity=10
- joint victor_right_gripper_fingerC_joint_2: limit lower=-1 upper=1 effort=300 velocity=10 -> lower=0 upper=1.2217304763960307 effort=300 velocity=10

File: urdf/victor_right_arm_with_rod.urdf.xacro (robot description, xacro)
@@ -4,7 +4,7 @@
     <link name="rod">
       <collision>
-        <origin xyz="0 0 0.05" rpy="0 0 0"/>
+        <origin xyz="0 0 0.0" rpy="0 0 0"/>
         <geometry>
-          <cylinder length="0.254" radius="0.03"/>
+          <cylinder length="0.234" radius="0.065"/>
         </geometry>
       </collision>
@@ -13,5 +13,5 @@
       <parent link="victor_right_gripper_palm"/>
       <child link="rod"/>
-      <origin xyz="0 0 0.1" rpy="1.57 0 0"/>
+      <origin xyz="0 0 0.15" rpy="1.57 0 0"/>
       <axis xyz="0 0 1"/>
     </joint>

Commit message: Changed to pringles can for real robot

File: urdf/victor_right_arm_with_rod.urdf (robot description, URDF)
Before this commit: robot victor_with_rod, 35 links, 34 joints
Links:
- link rod: geometry collision cylinder length=0.234 radius=0.038
Joints:
- joint rod_joint: origin xyz=0 0 0.15 rpy=1.57 0 0 -> xyz=0 0 0.0 rpy=0 0 0

File: urdf/victor_right_arm_with_rod.urdf.xacro (robot description, xacro)
@@ -2,9 +2,25 @@
 <robot name="victor_with_rod" xmlns:xacro="http://www.ros.org/wiki/xacro">
     <xacro:include filename="$(find gpu_voxel_planning)/urdf/victor_right_arm_only.urdf.xacro"/>
+    <!-- Pitcher -->
+    <!-- <link name="rod"> -->
+    <!--   <collision> -->
+    <!--     <origin xyz="0 0 -0.02" rpy="0 0 0"/> -->
+    <!--     <geometry> -->
+    <!--       <cylinder length="0.234" radius="0.065"/> -->
+    <!--     </geometry> -->
+    <!--   </collision> -->
+    <!-- </link> -->
+    <!-- <joint name="rod_joint" type="fixed"> -->
+    <!--   <parent link="victor_right_gripper_palm"/> -->
+    <!--   <child link="rod"/> -->
+    <!--   <origin xyz="0 0 0.15" rpy="1.57 0 0"/> -->
+    <!--   <axis xyz="0 0 1"/> -->
+    <!-- </joint> -->
+    <!-- Pringles -->
     <link name="rod">
       <collision>
-        <origin xyz="0 0 0.0" rpy="0 0 0"/>
+        <origin xyz="0 0 0.30" rpy="0 0 0"/>
         <geometry>
-          <cylinder length="0.234" radius="0.065"/>
+          <cylinder length="0.234" radius="0.038"/>
         </geometry>
       </collision>
@@ -13,5 +29,5 @@
       <parent link="victor_right_gripper_palm"/>
       <child link="rod"/>
-      <origin xyz="0 0 0.15" rpy="1.57 0 0"/>
+      <origin xyz="0 0 0.0" rpy="0 0 0"/>
       <axis xyz="0 0 1"/>
     </joint>

Commit message: Updated controller, checks all states now

File: urdf/victor_right_arm_with_rod.urdf (robot description, URDF)
Before this commit: robot victor_with_rod, 35 links, 34 joints
Links:
- link rod: geometry collision cylinder length=0.234 radius=0.065
Joints:
- joint rod_joint: origin xyz=0 0 0.0 rpy=0 0 0 -> xyz=0 0 0.15 rpy=1.57 0 0

File: urdf/victor_right_arm_with_rod.urdf.xacro (robot description, xacro)
@@ -3,9 +3,24 @@
     <xacro:include filename="$(find gpu_voxel_planning)/urdf/victor_right_arm_only.urdf.xacro"/>
     <!-- Pitcher -->
+    <link name="rod">
+      <collision>
+        <origin xyz="0 0 -0.02" rpy="0 0 0"/>
+        <geometry>
+          <cylinder length="0.234" radius="0.065"/>
+        </geometry>
+      </collision>
+    </link>
+    <joint name="rod_joint" type="fixed">
+      <parent link="victor_right_gripper_palm"/>
+      <child link="rod"/>
+      <origin xyz="0 0 0.15" rpy="1.57 0 0"/>
+      <axis xyz="0 0 1"/>
+    </joint>
+    <!-- Pringles -->
     <!-- <link name="rod"> -->
     <!--   <collision> -->
-    <!--     <origin xyz="0 0 -0.02" rpy="0 0 0"/> -->
+    <!--     <origin xyz="0 0 0.30" rpy="0 0 0"/> -->
     <!--     <geometry> -->
-    <!--       <cylinder length="0.234" radius="0.065"/> -->
+    <!--       <cylinder length="0.234" radius="0.038"/> -->
     <!--     </geometry> -->
     <!--   </collision> -->
@@ -14,21 +29,6 @@
     <!--   <parent link="victor_right_gripper_palm"/> -->
     <!--   <child link="rod"/> -->
-    <!--   <origin xyz="0 0 0.15" rpy="1.57 0 0"/> -->
+    <!--   <origin xyz="0 0 0.0" rpy="0 0 0"/> -->
     <!--   <axis xyz="0 0 1"/> -->
     <!-- </joint> -->
-    <!-- Pringles -->
-    <link name="rod">
-      <collision>
-        <origin xyz="0 0 0.30" rpy="0 0 0"/>
-        <geometry>
-          <cylinder length="0.234" radius="0.038"/>
-        </geometry>
-      </collision>
-    </link>
-    <joint name="rod_joint" type="fixed">
-      <parent link="victor_right_gripper_palm"/>
-      <child link="rod"/>
-      <origin xyz="0 0 0.0" rpy="0 0 0"/>
-      <axis xyz="0 0 1"/>
-    </joint>
 </robot>

Commit message: Added bar clamp

File: urdf/victor_right_arm_with_rod.urdf (robot description, URDF)
Before this commit: robot victor_with_rod, 35 links, 34 joints
Links:
- link rod: geometry collision mesh filename=package://gpu_voxel_planning/urdf/BarClamp_6in_scaled.stl scale=1 1 1
Joints:
- joint rod_joint: origin xyz=0 0 0.15 rpy=1.57 0 0 -> xyz=0 0 0.0 rpy=0 0 0

File: urdf/victor_right_arm_with_rod.urdf.xacro (robot description, xacro)
@@ -3,9 +3,25 @@
     <xacro:include filename="$(find gpu_voxel_planning)/urdf/victor_right_arm_only.urdf.xacro"/>
     <!-- Pitcher -->
+    <!-- <link name="rod"> -->
+    <!--   <collision> -->
+    <!--     <origin xyz="0 0 -0.02" rpy="0 0 0"/> -->
+    <!--     <geometry> -->
+    <!--       <cylinder length="0.234" radius="0.065"/> -->
+    <!--     </geometry> -->
+    <!--   </collision> -->
+    <!-- </link> -->
+    <!-- <joint name="rod_joint" type="fixed"> -->
+    <!--   <parent link="victor_right_gripper_palm"/> -->
+    <!--   <child link="rod"/> -->
+    <!--   <origin xyz="0 0 0.15" rpy="1.57 0 0"/> -->
+    <!--   <axis xyz="0 0 1"/> -->
+    <!-- </joint> -->
+    <!-- Clamp -->
     <link name="rod">
       <collision>
-        <origin xyz="0 0 -0.02" rpy="0 0 0"/>
+        <origin xyz="0 0 0.12" rpy="0 0 0"/>
         <geometry>
-          <cylinder length="0.234" radius="0.065"/>
+          <mesh filename="package://gpu_voxel_planning/urdf/BarClamp_6in_scaled.stl"
+                scale="1 1 1"/>
         </geometry>
       </collision>
@@ -14,5 +30,5 @@
       <parent link="victor_right_gripper_palm"/>
       <child link="rod"/>
-      <origin xyz="0 0 0.15" rpy="1.57 0 0"/>
+      <origin xyz="0 0 0.0" rpy="0 0 0"/>
       <axis xyz="0 0 1"/>
     </joint>

Commit message: table experiments

File: urdf/victor_right_arm_with_rod.urdf (robot description, URDF)
Before this commit: robot victor_with_rod, 35 links, 34 joints
Links:
- link rod: geometry collision cylinder length=0.234 radius=0.038
Joints:
- joint rod_joint: origin xyz=0 0 0.0 rpy=0 0 0 -> xyz=0 0 0.15 rpy=1.57 0 0

File: urdf/victor_right_arm_with_rod.urdf.xacro (robot description, xacro)
@@ -18,25 +18,10 @@
     <!-- </joint> -->
     <!-- Clamp -->
-    <link name="rod">
-      <collision>
-        <origin xyz="0 0 0.12" rpy="0 0 0"/>
-        <geometry>
-          <mesh filename="package://gpu_voxel_planning/urdf/BarClamp_6in_scaled.stl"
-                scale="1 1 1"/>
-        </geometry>
-      </collision>
-    </link>
-    <joint name="rod_joint" type="fixed">
-      <parent link="victor_right_gripper_palm"/>
-      <child link="rod"/>
-      <origin xyz="0 0 0.0" rpy="0 0 0"/>
-      <axis xyz="0 0 1"/>
-    </joint>
-    <!-- Pringles -->
     <!-- <link name="rod"> -->
     <!--   <collision> -->
-    <!--     <origin xyz="0 0 0.30" rpy="0 0 0"/> -->
+    <!--     <origin xyz="0 0 0.12" rpy="0 0 0"/> -->
     <!--     <geometry> -->
-    <!--       <cylinder length="0.234" radius="0.038"/> -->
+    <!--       <mesh filename="package://gpu_voxel_planning/urdf/BarClamp_6in_scaled.stl" -->
+    <!--             scale="1 1 1"/> -->
     <!--     </geometry> -->
     <!--   </collision> -->
@@ -48,3 +33,18 @@
     <!--   <axis xyz="0 0 1"/> -->
     <!-- </joint> -->
+    <!-- Pringles -->
+    <link name="rod">
+      <collision>
+        <origin xyz="0 0 -0.02" rpy="0 0 0"/>
+        <geometry>
+          <cylinder length="0.234" radius="0.038"/>
+        </geometry>
+      </collision>
+    </link>
+    <joint name="rod_joint" type="fixed">
+      <parent link="victor_right_gripper_palm"/>
+      <child link="rod"/>
+      <origin xyz="0 0 0.15" rpy="1.57 0 0"/>
+      <axis xyz="0 0 1"/>
+    </joint>
 </robot>

Commit message: Changes for this round of trials on real victor

File: urdf/victor_right_arm_with_rod.urdf (robot description, URDF)
Before this commit: robot victor_with_rod, 35 links, 34 joints
Links:
- link rod: geometry collision mesh filename=package://gpu_voxel_planning/urdf/BarClamp_6in_scaled.stl scale=1 1 1
Joints:
- joint rod_joint: origin xyz=0 0 0.15 rpy=1.57 0 0 -> xyz=0 0 0.0 rpy=0 0 0

File: urdf/victor_right_arm_with_rod.urdf.xacro (robot description, xacro)
@@ -18,10 +18,25 @@
     <!-- </joint> -->
     <!-- Clamp -->
+    <link name="rod">
+      <collision>
+        <origin xyz="0 0 0.12" rpy="0 0 0"/>
+        <geometry>
+          <mesh filename="package://gpu_voxel_planning/urdf/BarClamp_6in_scaled.stl"
+                scale="1 1 1"/>
+        </geometry>
+      </collision>
+    </link>
+    <joint name="rod_joint" type="fixed">
+      <parent link="victor_right_gripper_palm"/>
+      <child link="rod"/>
+      <origin xyz="0 0 0.0" rpy="0 0 0"/>
+      <axis xyz="0 0 1"/>
+    </joint>
+    <!-- Pringles -->
     <!-- <link name="rod"> -->
     <!--   <collision> -->
-    <!--     <origin xyz="0 0 0.12" rpy="0 0 0"/> -->
+    <!--     <origin xyz="0 0 -0.02" rpy="0 0 0"/> -->
     <!--     <geometry> -->
-    <!--       <mesh filename="package://gpu_voxel_planning/urdf/BarClamp_6in_scaled.stl" -->
-    <!--             scale="1 1 1"/> -->
+    <!--       <cylinder length="0.234" radius="0.038"/> -->
     <!--     </geometry> -->
     <!--   </collision> -->
@@ -30,21 +45,6 @@
     <!--   <parent link="victor_right_gripper_palm"/> -->
     <!--   <child link="rod"/> -->
-    <!--   <origin xyz="0 0 0.0" rpy="0 0 0"/> -->
+    <!--   <origin xyz="0 0 0.15" rpy="1.57 0 0"/> -->
     <!--   <axis xyz="0 0 1"/> -->
     <!-- </joint> -->
-    <!-- Pringles -->
-    <link name="rod">
-      <collision>
-        <origin xyz="0 0 -0.02" rpy="0 0 0"/>
-        <geometry>
-          <cylinder length="0.234" radius="0.038"/>
-        </geometry>
-      </collision>
-    </link>
-    <joint name="rod_joint" type="fixed">
-      <parent link="victor_right_gripper_palm"/>
-      <child link="rod"/>
-      <origin xyz="0 0 0.15" rpy="1.57 0 0"/>
-      <axis xyz="0 0 1"/>
-    </joint>
 </robot>

Commit message: Change goal location and a few other things for prepping for live demo

File: urdf/victor_right_arm_with_rod.urdf (robot description, URDF)
Before this commit: robot victor_with_rod, 35 links, 34 joints
Links:
- link rod: geometry collision cylinder length=0.234 radius=0.065
Joints:
- joint rod_joint: origin xyz=0 0 0.0 rpy=0 0 0 -> xyz=0 0 0.15 rpy=1.57 0 0

File: urdf/victor_right_arm_with_rod.urdf.xacro (robot description, xacro)
@@ -3,9 +3,25 @@
     <xacro:include filename="$(find gpu_voxel_planning)/urdf/victor_right_arm_only.urdf.xacro"/>
     <!-- Pitcher -->
+    <link name="rod">
+      <collision>
+        <origin xyz="0 0 -0.02" rpy="0 0 0"/>
+        <geometry>
+          <cylinder length="0.234" radius="0.065"/>
+        </geometry>
+      </collision>
+    </link>
+    <joint name="rod_joint" type="fixed">
+      <parent link="victor_right_gripper_palm"/>
+      <child link="rod"/>
+      <origin xyz="0 0 0.15" rpy="1.57 0 0"/>
+      <axis xyz="0 0 1"/>
+    </joint>
+    <!-- Clamp -->
     <!-- <link name="rod"> -->
     <!--   <collision> -->
-    <!--     <origin xyz="0 0 -0.02" rpy="0 0 0"/> -->
+    <!--     <origin xyz="0 0 0.12" rpy="0 0 0"/> -->
     <!--     <geometry> -->
-    <!--       <cylinder length="0.234" radius="0.065"/> -->
+    <!--       <mesh filename="package://gpu_voxel_planning/urdf/BarClamp_6in_scaled.stl" -->
+    <!--             scale="1 1 1"/> -->
     <!--     </geometry> -->
     <!--   </collision> -->
@@ -14,23 +30,7 @@
     <!--   <parent link="victor_right_gripper_palm"/> -->
     <!--   <child link="rod"/> -->
-    <!--   <origin xyz="0 0 0.15" rpy="1.57 0 0"/> -->
+    <!--   <origin xyz="0 0 0.0" rpy="0 0 0"/> -->
     <!--   <axis xyz="0 0 1"/> -->
     <!-- </joint> -->
-    <!-- Clamp -->
-    <link name="rod">
-      <collision>
-        <origin xyz="0 0 0.12" rpy="0 0 0"/>
-        <geometry>
-          <mesh filename="package://gpu_voxel_planning/urdf/BarClamp_6in_scaled.stl"
-                scale="1 1 1"/>
-        </geometry>
-      </collision>
-    </link>
-    <joint name="rod_joint" type="fixed">
-      <parent link="victor_right_gripper_palm"/>
-      <child link="rod"/>
-      <origin xyz="0 0 0.0" rpy="0 0 0"/>
-      <axis xyz="0 0 1"/>
-    </joint>
     <!-- Pringles -->
     <!-- <link name="rod"> -->
