Commit message: Added horrible hack to swap the left and right arms by swapping base links in the URDF

File: urdf/victor_left_arm_and_body.urdf (robot description, URDF)
Before this commit: robot victor, 34 links, 33 joints
Joints:
- removed joint victor_left_arm_mount_victor_left_arm_joint
- added joint victor_right_arm_mount_victor_left_arm_joint: type fixed, parent victor_right_arm_mount, child victor_left_arm_link_0, origin xyz=0 0 0 rpy=0 0 0
- joint gpu_voxel_world_joint: origin xyz=1.0 2.0 0.0 rpy=0.0 0.0 0.0 -> xyz=1.0 1.3 0.0 rpy=0.0 0.0 -0.7854
- joint victor_joint_left_arm_world_frame_kuka: parent victor_left_arm_mount -> victor_right_arm_mount
- joint victor_left_gripper_fingerA_joint_2: limit lower=-1 upper=1 effort=300 velocity=10 -> lower=0 upper=1.2217304763960307 effort=300 velocity=10
- joint victor_left_gripper_fingerB_joint_2: limit lower=-1 upper=1 effort=300 velocity=10 -> lower=0 upper=1.2217304763960307 effort=300 velocity=10
- joint victor_left_gripper_fingerC_joint_2: limit lower=-1 upper=1 effort=300 velocity=10 -> lower=0 upper=1.2217304763960307 effort=300 velocity=10

File: urdf/victor_left_arm_and_body.urdf.xacro (robot description, xacro)
@@ -14,9 +14,9 @@
     <!--Import the lbr iiwa macro -->
     <xacro:include filename="$(find gpu_voxel_planning)/urdf/iiwa7.xacro"/>
-    <xacro:iiwa7 hardware_interface="$(arg hardware_interface)" robot_name="$(arg robot_name)_left_arm" parent="$(arg robot_name)_left_arm_mount">
+    <xacro:iiwa7 hardware_interface="$(arg hardware_interface)" robot_name="$(arg robot_name)_left_arm" parent="$(arg robot_name)_right_arm_mount">
         <origin xyz="0 0 0" rpy="0 0 0"/>
     </xacro:iiwa7>
     <joint name="$(arg robot_name)_joint_left_arm_world_frame_kuka" type="fixed">
-        <parent link="$(arg robot_name)_left_arm_mount"/>
+        <parent link="$(arg robot_name)_right_arm_mount"/>
         <child link="$(arg robot_name)_left_arm_world_frame_kuka"/>
         <origin xyz="0 0 0" rpy="1.57079632679 0 0"/>
@@ -54,8 +54,13 @@
     <!-- </xacro:robotiq_3finger> -->
     <link name="gpu_voxel_world"/>
+    <!-- <joint name="gpu_voxel_world_joint" type="fixed"> -->
+    <!--   <parent link="gpu_voxel_world"/> -->
+    <!--   <child link="victor_root"/> -->
+    <!--   <origin rpy="0.0 0.0 0.0" xyz="1.0 2.0 0.0"/> -->
+    <!-- </joint> -->
     <joint name="gpu_voxel_world_joint" type="fixed">
       <parent link="gpu_voxel_world"/>
       <child link="victor_root"/>
-      <origin rpy="0.0 0.0 0.0" xyz="1.0 2.0 0.0"/>
+      <origin rpy="0.0 0.0 -0.7854" xyz="1.0 1.3 0.0"/>
     </joint>
 </robot>

File: urdf/victor_right_arm_and_body.urdf.xacro (robot description, xacro)
@@ -24,11 +24,11 @@
     <!-- <link name="$(arg robot_name)_left_arm_world_frame_kuka"> -->
     <!-- </link> -->
-    <xacro:iiwa7 hardware_interface="$(arg hardware_interface)" robot_name="$(arg robot_name)_right_arm" parent="$(arg robot_name)_right_arm_mount">
+    <xacro:iiwa7 hardware_interface="$(arg hardware_interface)" robot_name="$(arg robot_name)_right_arm" parent="$(arg robot_name)_left_arm_mount">
         <origin xyz="0 0 0" rpy="0 0 0"/>
     </xacro:iiwa7>
     <joint name="$(arg robot_name)_joint_right_arm_world_frame_kuka" type="fixed">
-        <parent link="$(arg robot_name)_right_arm_mount"/>
+        <parent link="$(arg robot_name)_left_arm_mount"/>
         <child link="$(arg robot_name)_right_arm_world_frame_kuka"/>
-        <origin xyz="0 0 0" rpy="-1.57079632679 0 0"/>
+        <origin xyz="0 0 0" rpy="1.57079632679 0 0"/>
     </joint>
     <link name="$(arg robot_name)_right_arm_world_frame_kuka">

File: urdf/victor_right_arm_only.urdf (robot description, URDF)
Before this commit: robot victor, 34 links, 33 joints
Joints:
- removed joint victor_right_arm_mount_victor_right_arm_joint
- added joint victor_left_arm_mount_victor_right_arm_joint: type fixed, parent victor_left_arm_mount, child victor_right_arm_link_0, origin xyz=0 0 0 rpy=0 0 0
- joint gpu_voxel_world_joint: origin xyz=1.0 2.0 0.0 rpy=0.0 0.0 0.0 -> xyz=1.0 1.3 0.0 rpy=0.0 0.0 -0.7854
- joint victor_joint_right_arm_world_frame_kuka: parent victor_right_arm_mount -> victor_left_arm_mount
- joint victor_right_gripper_fingerA_joint_2: limit lower=-1 upper=1 effort=300 velocity=10 -> lower=0 upper=1.2217304763960307 effort=300 velocity=10
- joint victor_right_gripper_fingerB_joint_2: limit lower=-1 upper=1 effort=300 velocity=10 -> lower=0 upper=1.2217304763960307 effort=300 velocity=10
- joint victor_right_gripper_fingerC_joint_2: limit lower=-1 upper=1 effort=300 velocity=10 -> lower=0 upper=1.2217304763960307 effort=300 velocity=10

File: urdf/victor_right_arm_only.urdf.xacro (robot description, xacro)
@@ -24,9 +24,9 @@
     <!-- <link name="$(arg robot_name)_left_arm_world_frame_kuka"> -->
     <!-- </link> -->
-    <xacro:iiwa7 hardware_interface="$(arg hardware_interface)" robot_name="$(arg robot_name)_right_arm" parent="$(arg robot_name)_right_arm_mount">
+    <xacro:iiwa7 hardware_interface="$(arg hardware_interface)" robot_name="$(arg robot_name)_right_arm" parent="$(arg robot_name)_left_arm_mount">
         <origin xyz="0 0 0" rpy="0 0 0"/>
     </xacro:iiwa7>
     <joint name="$(arg robot_name)_joint_right_arm_world_frame_kuka" type="fixed">
-        <parent link="$(arg robot_name)_right_arm_mount"/>
+        <parent link="$(arg robot_name)_left_arm_mount"/>
         <child link="$(arg robot_name)_right_arm_world_frame_kuka"/>
         <origin xyz="0 0 0" rpy="-1.57079632679 0 0"/>
@@ -54,8 +54,13 @@
     </xacro:robotiq_3finger>
     <link name="gpu_voxel_world"/>
+    <!-- <joint name="gpu_voxel_world_joint" type="fixed"> -->
+    <!--   <parent link="gpu_voxel_world"/> -->
+    <!--   <child link="victor_root"/> -->
+    <!--   <origin rpy="0.0 0.0 0.0" xyz="1.0 2.0 0.0"/> -->
+    <!-- </joint> -->
     <joint name="gpu_voxel_world_joint" type="fixed">
       <parent link="gpu_voxel_world"/>
       <child link="victor_root"/>
-      <origin rpy="0.0 0.0 0.0" xyz="1.0 2.0 0.0"/>
+      <origin rpy="0.0 0.0 -0.7854" xyz="1.0 1.3 0.0"/>
     </joint>
 </robot>
