Commit message: Moved strategies to separate folder

File: urdf/victor.urdf.xacro (robot description, xacro)
@@ -53,3 +53,9 @@
         <origin xyz="0 0 0.02705" rpy="0 0 ${PI/4}"/> <!-- Offset measured with a tape measure; please confirm/fix this value -->
     </xacro:robotiq_3finger>
+    <link name="gpu_voxel_world"/>
+    <joint name="gpu_voxel_world_joint" type="fixed">
+      <parent link="gpu_voxel_world"/>
+      <child link="victor_root"/>
+      <origin rpy="0.0 0.0 0.0" xyz="1.0 2.0 0.0"/>
+    </joint>
 </robot>

Commit message: Update to work with Peters new moveit arm_robots

File: urdf/victor.urdf.xacro (robot description, xacro)
@@ -1,7 +1,8 @@
 <?xml version="1.0"?>
 <robot name="victor" xmlns:xacro="http://www.ros.org/wiki/xacro">
+    <xacro:property name="gripper" value="kinematic_robotiq" />
     <xacro:arg name="robot_name" default="victor"/>
-    <xacro:arg name="hardware_interface" default="PositionJointInterface"/>
-        <!-- Import Rviz colors -->
+    <xacro:arg name="hardware_interface" default="hardware_interface/PositionJointInterface"/>
+    <!-- Import Rviz colors -->
     <xacro:include filename="$(find victor_description)/urdf/materials.xacro"/>
     <!-- pedestal -->
@@ -14,5 +15,6 @@
     <!--Import the lbr iiwa macro -->
     <xacro:include filename="$(find victor_description)/urdf/iiwa7.xacro"/>
-    <xacro:iiwa7 hardware_interface="$(arg hardware_interface)" robot_name="$(arg robot_name)_left_arm" parent="$(arg robot_name)_left_arm_mount">
+    <xacro:iiwa7 hardware_interface="$(arg hardware_interface)" robot_name="$(arg robot_name)_left_arm"
+                 parent="$(arg robot_name)_left_arm_mount">
         <origin xyz="0 0 0" rpy="0 0 0"/>
     </xacro:iiwa7>
@@ -24,5 +26,6 @@
     <link name="$(arg robot_name)_left_arm_world_frame_kuka">
     </link>
-    <xacro:iiwa7 hardware_interface="$(arg hardware_interface)" robot_name="$(arg robot_name)_right_arm" parent="$(arg robot_name)_right_arm_mount">
+    <xacro:iiwa7 hardware_interface="$(arg hardware_interface)" robot_name="$(arg robot_name)_right_arm"
+                 parent="$(arg robot_name)_right_arm_mount">
         <origin xyz="0 0 0" rpy="0 0 0"/>
     </xacro:iiwa7>
@@ -37,20 +40,25 @@
     <xacro:include filename="$(find victor_description)/urdf/iiwa7_to_robotiq_adapter.xacro"/>
     <xacro:iia7_to_robotiq_adapter parent="$(arg robot_name)_left_arm_flange" prefix="$(arg robot_name)_left">
-        <!--<origin xyz="0 0 0" rpy="${PI/2} 0 ${PI/4}"/> &lt;!&ndash; Offset measured with a tape measure; please confirm/fix this value &ndash;&gt;-->
-        <origin xyz="0 0 0" rpy="0 0 0"/>
+        <origin xyz="0 0 -0.01" rpy="0 0 0"/>
     </xacro:iia7_to_robotiq_adapter>
     <xacro:iia7_to_robotiq_adapter parent="$(arg robot_name)_right_arm_flange" prefix="$(arg robot_name)_right">
-        <!--<origin xyz="0 0 0" rpy="${PI/2} 0 ${PI/4}"/> &lt;!&ndash; Offset measured with a tape measure; please confirm/fix this value &ndash;&gt;-->
-        <origin xyz="0 0 0" rpy="0 0 0"/>
+        <origin xyz="0 0 -0.01" rpy="0 0 0"/>
     </xacro:iia7_to_robotiq_adapter>
     <!-- Robotiq grippers -->
-    <!--Import the Robotiq 3 finger macro -->
-    <xacro:include filename="$(find victor_description)/urdf/robotiq_3finger_gripper.xacro"/>
-    <xacro:robotiq_3finger parent="$(arg robot_name)_left_gripper_mounting_bracket" prefix="$(arg robot_name)_left_gripper">
-        <origin xyz="0 0 0.02705" rpy="0 0 ${PI/4}"/> <!-- Offset measured with a tape measure; please confirm/fix this value -->
-    </xacro:robotiq_3finger>
-    <xacro:robotiq_3finger parent="$(arg robot_name)_right_gripper_mounting_bracket" prefix="$(arg robot_name)_right_gripper">
-        <origin xyz="0 0 0.02705" rpy="0 0 ${PI/4}"/> <!-- Offset measured with a tape measure; please confirm/fix this value -->
-    </xacro:robotiq_3finger>
+    <xacro:if value="${gripper == 'kinematic_robotiq'}">
+        <xacro:include filename="$(find victor_description)/urdf/kinematic_robotiq_grippers.xacro"/>
+    </xacro:if>
+    <xacro:if value="${gripper == 'robotiq'}">
+        <xacro:include filename="$(find victor_description)/urdf/robotiq_grippers.xacro"/>
+    </xacro:if>
+    <!-- Define additional links as "tools", which are useful for planning and getting transforms -->
+    <xacro:include filename="$(find victor_description)/urdf/robotiq_pinch_grasp_tools.xacro"/>
+    <xacro:robotiq_pinch_grasp_tools robot_name="$(arg robot_name)"/>
+    <!-- Add Gazebo properties for whole robot -->
+    <xacro:include filename="$(find victor_description)/urdf/victor.gazebo.xacro"/>
+    <xacro:include filename="$(find victor_description)/urdf/gazebo_utilities.xacro"/>
+    <!-- Load Gazebo lib and set the robot namespace -->
+    <xacro:add_gazebo_control_plugin robot_namespace="$(arg robot_name)"/>
+    <!-- <xacro:add_moveit_planning_scene_plugin robot_namespace="$(arg robot_name)" root_frame_id="victor_root"/> -->
     <link name="gpu_voxel_world"/>
     <joint name="gpu_voxel_world_joint" type="fixed">
